File: HCPL-7840.brd (EAGLE design)
At the start: 52 parts, among them J1 0

Commit message: .
Parts:
- added RS: R, 75ShS:75ШС
- C8: device rcl:C0805 -> rcl:C075-032X103
- R11: value 1 -> (none)
- moved GND7 21.6 mm to (27.6, 23.2)
- moved L4 17.2 mm to (-11.4, 33.7)
- moved DA5 14.9 mm to (7.62, 23.8)
- moved C13 14.6 mm to (0.95, 38.4)
- moved C18 14.6 mm to (14.3, 25.4)
- moved VD1 14.6 mm to (16.5, 35.9)
- moved C19 14.6 mm to (3.49, 25.1)
- moved +12V 14.6 mm to (18.7, 31.8)
- moved C11 14.6 mm to (8.57, 39.1)
- moved C12 14.6 mm to (10.8, 39.1)
- moved DA4 14.6 mm to (5.40, 33.7)
- moved GND 14.6 mm to (18.7, 26.7)
- moved L1 14.6 mm to (-5.40, 35.2)
- moved R10 14.6 mm to (14.3, 31.8)
- moved R11 14.6 mm to (11.1, 33.0)
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Routing:
- net GND: track 174.2 -> 161.4 mm
- net N$16: track 10.9 -> 0.00 mm
- net N$12: track 6.71 -> 1.95 mm
- net +5V: track 17.6 -> 22.1 mm
- net N$5: track 10.6 -> 13.2 mm
- net N$9: track 7.36 -> 9.79 mm
- net V-: track 4.76 -> 6.67 mm
- net N$8: track 19.2 -> 20.3 mm
- net N$13: track 2.79 -> 2.21 mm

Commit message: .
Parts:
- moved C3 14.3 mm to (-6.67, 1.91)
- moved RS 7.16 mm to (-13.3, -2.54), turned to 180 degrees
- moved R5 6.70 mm to (-19.4, 3.17), turned to 90 degrees
Connections:
- net R_SENSE: now also RS.P$2
- net V-: now also RS.P$1
Changed lines of the file:
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@@
 <board>
 <plain>
-<dimension x1="-42.2275" y1="-27.94" x2="30.1625" y2="-26.035" x3="-6.0325" y3="58.42" textsize="1.778" layer="21" dtype="horizontal"/>
+<dimension x1="-42.2275" y1="-27.94" x2="22.225" y2="-24.765" x3="-10.00125" y3="58.42" textsize="1.778" layer="21" dtype="horizontal"/>
 <dimension x1="57.4675" y1="43.815" x2="56.515" y2="-20.0025" x3="-54.9275" y3="11.90625" textsize="1.778" layer="21" dtype="vertical"/>
 <circle x="1.905" y="32.7025" radius="5" width="0.6096" layer="21"/>
@@
 <circle x="35.8775" y="23.1775" radius="2.5" width="0.1" layer="21"/>
 <circle x="33.3375" y="18.7325" radius="2.5" width="0.1" layer="21"/>
-<circle x="34.29" y="18.0975" radius="2.5" width="0.1" layer="21"/>
+<circle x="10.795" y="8.89" radius="2.5" width="0.1" layer="21"/>
 <circle x="-43.18" y="35.8775" radius="2.5" width="0.1" layer="21"/>
 <circle x="-41.5925" y="23.495" radius="2.5" width="0.1" layer="21"/>
@@
 </autorouter>
 <elements>
-<element name="R5" library="rcl" package="M0805" value="39" x="-26.035" y="2.54" rot="MR180"/>
+<element name="R5" library="rcl" package="M0805" value="39" x="-19.3675" y="3.175" rot="MR90"/>
 <element name="DA2" library="linear" package="SO08" value="LM358D" x="11.43" y="15.24" rot="MR270"/>
 <element name="DA4" library="MC34063" package="SOIC8" value="MC34063AD" x="5.3975" y="33.655" rot="MR90"/>
-<element name="C3" library="rcl" package="C0805" value="10n" x="-20.955" y="2.54" rot="MR180"/>
+<element name="C3" library="rcl" package="C0805" value="10n" x="-6.6675" y="1.905" rot="MR180"/>
 <element name="C2" library="rcl" package="C075-032X103" value="100n" x="-22.86" y="15.24" rot="R270"/>
 <element name="DA1" library="avago" package="DIL08" value="HCPL-7800" x="-16.8275" y="15.24" rot="R270">
@@
 <element name="GND8" library="Разъёмы штырьковые 2.54мм" package="1X01" value="" x="30.7975" y="27.305"/>
 <element name="R10" library="rcl" package="M1206" value="1" x="14.2875" y="31.75" rot="MR270"/>
-<element name="RS" library="75ShS" package="75ШС" value="R" x="-6.35" y="-0.9525"/>
+<element name="RS" library="75ShS" package="75ШС" value="R" x="-13.335" y="-2.54" rot="R180"/>
 </elements>
 <signals>
 <signal name="R_SENSE">
 <contactref element="R5" pad="1"/>
+<contactref element="RS" pad="P$2"/>
+<wire x1="-19.3675" y1="2.225" x2="-34.335" y2="1.46" width="0" layer="19" extent="16-16"/>
 </signal>
 <signal name="N$1">
@@
 <wire x1="-20.6375" y1="16.51" x2="-25.4" y2="16.51" width="0.6096" layer="16"/>
 <wire x1="-25.4" y1="16.51" x2="-25.4" y2="10.16" width="0.6096" layer="16"/>
-<wire x1="-21.905" y1="2.54" x2="-25.085" y2="2.54" width="0" layer="19" extent="16-16"/>
-<wire x1="-25.4" y1="10.16" x2="-25.085" y2="2.54" width="0" layer="19" extent="16-16"/>
+<wire x1="-7.6175" y1="1.905" x2="-19.3675" y2="4.125" width="0" layer="19" extent="16-16"/>
+<wire x1="-25.4" y1="10.16" x2="-19.3675" y2="4.125" width="0" layer="19" extent="16-16"/>
 </signal>
 <signal name="N$2">
@@
 <wire x1="-20.6375" y1="13.97" x2="-20.6375" y2="11.43" width="1.27" layer="16"/>
 <wire x1="-14.605" y1="32.7025" x2="-16.51" y2="32.7025" width="0.6096" layer="16"/>
+<contactref element="RS" pad="P$1"/>
 <wire x1="-14.605" y1="32.7025" x2="-8.5725" y2="31.79" width="0" layer="19" extent="16-16"/>
 <wire x1="-18.745" y1="30.48" x2="-16.51" y2="32.7025" width="0" layer="19" extent="16-16"/>
@@
 <wire x1="-19.6825" y1="39.6875" x2="-20.64" y2="37.465" width="0" layer="19" extent="16-16"/>
 <wire x1="-20.6375" y1="13.97" x2="-21.412" y2="30.48" width="0" layer="19" extent="16-16"/>
-<wire x1="-20.005" y1="2.54" x2="-20.6375" y2="11.43" width="0" layer="19" extent="16-16"/>
+<wire x1="-5.7175" y1="1.905" x2="-20.6375" y2="11.43" width="0" layer="19" extent="16-16"/>
+<wire x1="7.665" y1="1.46" x2="-5.7175" y2="1.905" width="0" layer="19" extent="16-16"/>
 </signal>
 <signal name="N$16">

Commit message: .
Parts:
- R1, R2: value 1k00 -> 10k
Changed lines of the file:
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@@
 <element name="L4" library="rcl" package="0204/7" value="" x="-11.43" y="33.655" rot="R270"/>
 <element name="C19" library="rcl" package="C0805" value="100n" x="3.4925" y="25.0825" rot="MR270"/>
-<element name="R2" library="rcl" package="M0805" value="1k00" x="-6.0325" y="18.7325" rot="MR180"/>
-<element name="R1" library="rcl" package="M0805" value="1k00" x="-6.0325" y="11.7475" rot="MR180"/>
+<element name="R2" library="rcl" package="M0805" value="10k" x="-6.0325" y="18.7325" rot="MR180"/>
+<element name="R1" library="rcl" package="M0805" value="10k" x="-6.0325" y="11.7475" rot="MR180"/>
 <element name="C17" library="rcl" package="C0805" value="100n" x="-11.43" y="40.64" rot="MR90"/>
 <element name="DA5" library="linear" package="SOT89" value="78L05F" x="7.62" y="23.8125" rot="MR90"/>
